Commit message: Start finishing phase. Finished the last open functions for the WBM-Class, removed some bugs and made several variable renamings (removed 'rlnk' and 'rootLnk').

File: mex-wholebodymodel/matlab/wrappers/+WBM/+Robot/+iCub_arms_torso_free/model_arms_torso_free.urdf (robot description, URDF)
Before this commit: robot iCub, 56 links, 55 joints
Joints:
- joint l_elbow: limit lower=0.0959931 upper=1.85005 effort=20 velocity=100 -> lower=0.2618 upper=1.4835 effort=20 velocity=100
- joint l_shoulder_pitch: limit lower=-1.65806 upper=0.0872665 effort=84 velocity=100 -> lower=-1.4835 upper=0.1047 effort=84 velocity=100
- joint l_shoulder_roll: limit lower=0 upper=2.80649 effort=84 velocity=100 -> lower=0.2618 upper=1.3963 effort=84 velocity=100
- joint l_shoulder_yaw: limit lower=-0.645772 upper=1.74533 effort=34 velocity=100 -> lower=-0.2618 upper=1.3614 effort=34 velocity=100
- joint l_wrist_pitch: limit lower=-1.13446 upper=0.174533 effort=0.65 velocity=100 -> lower=-1.2217 upper=0.0000 effort=0.65 velocity=100
- joint l_wrist_prosup: limit lower=-0.872665 upper=0.872665 effort=0.45 velocity=100 -> lower=-1.2217 upper=1.0472 effort=0.45 velocity=100
- joint l_wrist_yaw: limit lower=-0.436332 upper=0.436332 effort=0.65 velocity=100 -> lower=-0.1745 upper=0.5236 effort=0.65 velocity=100
- joint r_elbow: limit lower=0.0959931 upper=1.85005 effort=20 velocity=100 -> lower=0.2618 upper=1.4835 effort=20 velocity=100
- joint r_shoulder_pitch: limit lower=-1.65806 upper=0.0872665 effort=84 velocity=100 -> lower=-1.4835 upper=0.1047 effort=84 velocity=100
- joint r_shoulder_roll: limit lower=0 upper=2.80649 effort=84 velocity=100 -> lower=0.2618 upper=1.3963 effort=84 velocity=100
- joint r_shoulder_yaw: limit lower=-0.645772 upper=1.74533 effort=34 velocity=100 -> lower=-0.2618 upper=1.3614 effort=34 velocity=100
- joint r_wrist_pitch: limit lower=-1.13446 upper=0.174533 effort=0.65 velocity=100 -> lower=-1.2217 upper=0.000 effort=0.65 velocity=100
- joint r_wrist_prosup: limit lower=-0.872665 upper=0.872665 effort=0.45 velocity=100 -> lower=-1.2217 upper=1.0472 effort=0.45 velocity=100
- joint r_wrist_yaw: limit lower=-0.436332 upper=0.436332 effort=0.65 velocity=100 -> lower=-0.1745 upper=0.5236 effort=0.65 velocity=100
- joint torso_pitch: limit lower=-0.383972 upper=1.46608 effort=36 velocity=100 -> lower=-0.3491 upper=1.2217 effort=36 velocity=100
- joint torso_roll: limit lower=-0.680678 upper=0.680678 effort=80 velocity=100 -> lower=-0.5236 upper=0.5236 effort=80 velocity=100
- joint torso_yaw: limit lower=-1.02974 upper=1.02974 effort=80 velocity=100 -> lower=-0.8727 upper=0.8727 effort=80 velocity=100
