Commit message: further simplifications for visualization

File: controllers/models/walkman/model.urdf (robot description, URDF)
Before this commit: robot bigman, 85 links, 84 joints
Links:
- link TorsoProtections: geometry collision mesh filename=meshes/simple/ProtectionSystem.STL scale=0.001 0.001 0.001
- link multisense/hokuyo_link: geometry collision box size=0.08 0.06 0.04238; collision cylinder length=0.047 radius=0.024425

Commit message: fixed visualization for walkman. meshes total size reduced from 25 to 6 Mb

File: controllers/models/walkman/model.urdf (robot description, URDF)
Before this commit: robot bigman, 85 links, 84 joints
Links:
- link DWL: geometry collision mesh filename=meshes/collision/TorsoRoll.STL scale=0.001 0.001 0.001; visual mesh filename=meshes/visual/TorsoRoll.dae scale=0.001 0.001 0.001
- link DWS: geometry collision mesh filename=meshes/collision/TorsoYawPitch.STL scale=0.001 0.001 0.001; visual mesh filename=meshes/visual/TorsoYawPitch.dae scale=0.001 0.001 0.001
- link DWYTorso: geometry collision mesh filename=meshes/collision/NewChest.STL scale=0.001 0.001 0.001; visual mesh filename=meshes/visual/NewChest.dae scale=0.001 0.001 0.001
- link LElb: geometry collision mesh filename=meshes/collision/Elbow.STL scale=0.001 -0.001 0.001; visual mesh filename=meshes/visual/Elbow.dae scale=0.001 -0.001 0.001
- link LFoot: geometry collision box size=0.32 0.16 0.015; visual mesh filename=meshes/visual/NewFoot.dae scale=0.001 -0.001 0.001
- link LFootmot: geometry collision mesh filename=meshes/collision/AnklePitch.STL scale=0.001 -0.001 0.001; visual mesh filename=meshes/visual/AnklePitch.dae scale=0.001 -0.001 0.001
- link LForearm: geometry collision mesh filename=meshes/collision/Forearm.STL scale=0.001 -0.001 0.001; visual mesh filename=meshes/visual/Forearm.dae scale=0.001 -0.001 0.001
- link LHipMot: geometry collision mesh filename=meshes/collision/HipRoll.STL scale=0.001 -0.001 0.001; visual mesh filename=meshes/visual/HipRoll.dae scale=0.001 -0.001 0.001
- link LLowLeg: geometry collision mesh filename=meshes/collision/KneePitchCalf.STL scale=0.001 -0.001 0.001; visual mesh filename=meshes/visual/KneePitchCalf.dae scale=0.001 -0.001 0.001
- link LShp: geometry collision mesh filename=meshes/collision/ShoulderPitch.STL scale=0.001 -0.001 0.001; visual mesh filename=meshes/visual/ShoulderPitch.dae scale=0.001 -0.001 0.001
- link LShr: geometry collision mesh filename=meshes/collision/TopUpperArm.STL scale=0.001 -0.001 0.001; visual mesh filename=meshes/visual/TopUpperArm.dae scale=0.001 -0.001 0.001
- link LShy: geometry collision mesh filename=meshes/collision/BottomUpperArm.STL scale=0.001 -0.001 0.001; visual mesh filename=meshes/visual/BottomUpperArm.dae scale=0.001 -0.001 0.001
- link LSoftHandLink: geometry collision mesh filename=meshes/collision/SoftHandOpen.STL scale=0.001 -0.001 0.001; visual mesh filename=meshes/visual/SoftHandOpen.dae scale=0.001 -0.001 0.001
- link LThighLowLeg: geometry collision mesh filename=meshes/collision/HipPitch.STL scale=0.001 -0.001 0.001; visual mesh filename=meshes/visual/HipPitch.dae scale=0.001 -0.001 0.001
- link LThighUpLeg: geometry collision mesh filename=meshes/collision/HipYaw.STL scale=0.001 -0.001 0.001; visual mesh filename=meshes/visual/HipYaw.dae scale=0.001 -0.001 0.001
- link LWrMot2: geometry collision mesh filename=meshes/collision/ForearmPitch.STL scale=0.001 -0.001 0.001; visual mesh filename=meshes/visual/ForearmPitch.dae scale=0.001 -0.001 0.001
- link LWrMot3: geometry collision mesh filename=meshes/collision/ForearmRoll.STL scale=0.001 -0.001 0.001; visual mesh filename=meshes/visual/ForearmRoll.dae scale=0.001 -0.001 0.001
- link NeckPitch: geometry collision mesh filename=meshes/collision/NeckPitch.STL scale=0.001 0.001 0.001; visual mesh filename=meshes/visual/NeckPitch.dae scale=0.001 0.001 0.001
- link NeckYaw: geometry collision mesh filename=meshes/collision/NeckYaw.STL scale=0.001 0.001 0.001; visual mesh filename=meshes/visual/NeckYaw.dae scale=0.001 0.001 0.001
- link RElb: geometry collision mesh filename=meshes/collision/Elbow.STL scale=0.001 0.001 0.001; visual mesh filename=meshes/visual/Elbow.dae scale=0.001 0.001 0.001
- link RFoot: geometry collision box size=0.32 0.16 0.015; visual mesh filename=meshes/visual/NewFoot.dae scale=0.001 0.001 0.001
- link RFootmot: geometry collision mesh filename=meshes/collision/AnklePitch.STL scale=0.001 0.001 0.001; visual mesh filename=meshes/visual/AnklePitch.dae scale=0.001 0.001 0.001
- link RForearm: geometry collision mesh filename=meshes/collision/Forearm.STL scale=0.001 0.001 0.001; visual mesh filename=meshes/visual/Forearm.dae scale=0.001 0.001 0.001
- link RHipMot: geometry collision mesh filename=meshes/collision/HipRoll.STL scale=0.001 0.001 0.001; visual mesh filename=meshes/visual/HipRoll.dae scale=0.001 0.001 0.001
- link RLowLeg: geometry collision mesh filename=meshes/collision/KneePitchCalf.STL scale=0.001 0.001 0.001; visual mesh filename=meshes/visual/KneePitchCalf.dae scale=0.001 0.001 0.001
- link RShp: geometry collision mesh filename=meshes/collision/ShoulderPitch.STL scale=0.001 0.001 0.001; visual mesh filename=meshes/visual/ShoulderPitch.dae scale=0.001 0.001 0.001
- link RShr: geometry collision mesh filename=meshes/collision/TopUpperArm.STL scale=0.001 0.001 0.001; visual mesh filename=meshes/visual/TopUpperArm.dae scale=0.001 0.001 0.001
- link RShy: geometry collision mesh filename=meshes/collision/BottomUpperArm.STL scale=0.001 0.001 0.001; visual mesh filename=meshes/visual/BottomUpperArm.dae scale=0.001 0.001 0.001
- link RSoftHandLink: geometry collision mesh filename=meshes/collision/SoftHandOpen.STL scale=0.001 0.001 0.001; visual mesh filename=meshes/visual/SoftHandOpen.dae scale=0.001 0.001 0.001
- link RThighLowLeg: geometry collision mesh filename=meshes/collision/HipPitch.STL scale=0.001 0.001 0.001; visual mesh filename=meshes/visual/HipPitch.dae scale=0.001 0.001 0.001
- link RThighUpLeg: geometry collision mesh filename=meshes/collision/HipYaw.STL scale=0.001 0.001 0.001; visual mesh filename=meshes/visual/HipYaw.dae scale=0.001 0.001 0.001
- link RWrMot2: geometry collision mesh filename=meshes/scollision/ForearmPitch.STL scale=0.001 0.001 0.001; visual mesh filename=meshes/visual/ForearmPitch.dae scale=0.001 0.001 0.001
- link RWrMot3: geometry collision mesh filename=meshes/collision/ForearmRoll.STL scale=0.001 0.001 0.001; visual mesh filename=meshes/visual/ForearmRoll.dae scale=0.001 0.001 0.001
- link TorsoProtections: geometry collision mesh filename=meshes/collision/ProtectionSystem.STL scale=0.001 0.001 0.001
- link Waist: geometry collision mesh filename=meshes/collision/Waist.STL scale=0.001 0.001 0.001; visual mesh filename=meshes/visual/Waist.dae scale=0.001 0.001 0.001
- link multisense/head: geometry collision mesh filename=meshes/collision/Head.STL scale=0.001 0.001 0.001; visual mesh filename=meshes/visual/Head.dae scale=0.001 0.001 0.001

Commit message: updated walkman meshes

File: controllers/models/walkman/model.urdf (robot description, URDF)
Before this commit: robot bigman, 85 links, 84 joints
Links:
- link TorsoProtections: geometry collision mesh filename=meshes/collision/ProtectionSystem.STL scale=0.001 0.001 0.001; visual mesh filename=/meshes/visual/ProtectionSystem.dae scale=0.001 0.001 0.001
